File: MRCS-ODX4.brd (EAGLE design)
At the start: 97.8 x 68.6 mm, 15 parts

Commit message: V1.7
moved 5mm connectors, updated labels, added power LEDs
Routing:
- net VIN: track 0.00 -> 118.1 mm
- net S$10: track 102.9 -> 0.00 mm
- net GND: track 0.00 -> 64.1 mm
- net S$12: track 54.6 -> 0.00 mm
- net S$15: track 15.2 -> 0.00 mm
- net S$7: track 9.53 -> 0.00 mm
Changed lines of the file:
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@@
 <?xml version="1.0" encoding="utf-8"?>
 <!DOCTYPE eagle SYSTEM "eagle.dtd">
-<eagle version="6.5.0">
+<eagle version="7.7.0">
 <drawing>
 <settings>
@@
 <setting verticaltext="up"/>
 </settings>
-<grid distance="0.025" unitdist="inch" unit="inch" style="lines" multiple="1" display="yes" altdistance="0.025" altunitdist="inch" altunit="inch"/>
+<grid distance="50" unitdist="mil" unit="mil" style="dots" multiple="2" display="yes" altdistance="25" altunitdist="mil" altunit="mil"/>
 <layers>
 <layer number="1" name="Top" color="4" fill="1" visible="yes" active="yes"/>
@@
 <pass name="Default">
 <param name="RoutingGrid" value="50mil"/>
+<param name="AutoGrid" value="1"/>
+<param name="Efforts" value="0"/>
+<param name="TopRouterVariant" value="1"/>
 <param name="tpViaShape" value="round"/>
 <param name="PrefDir.1" value="|"/>
@@
 <wire x1="69.85" y1="50.8" x2="69.85" y2="45.72" width="1.27" layer="16"/>
 </signal>
-<signal name="S$7">
-<wire x1="66.04" y1="46.355" x2="66.04" y2="55.88" width="0.6096" layer="1"/>
-</signal>
-<signal name="S$12">
-<wire x1="16.51" y1="48.26" x2="66.04" y2="48.26" width="0.6096" layer="16"/>
-<wire x1="16.51" y1="48.26" x2="16.51" y2="45.72" width="0.6096" layer="16"/>
-<wire x1="66.04" y1="48.26" x2="66.04" y2="45.72" width="0.6096" layer="16"/>
-</signal>
 <signal name="S$14">
 <wire x1="66.04" y1="11.43" x2="66.04" y2="13.97" width="0.6096" layer="16"/>
 <wire x1="16.51" y1="11.43" x2="66.04" y2="11.43" width="0.6096" layer="16"/>
 <wire x1="16.51" y1="11.43" x2="16.51" y2="13.97" width="0.6096" layer="16"/>
-</signal>
-<signal name="S$10">
-<wire x1="24.13" y1="16.51" x2="24.13" y2="19.05" width="0.6096" layer="16"/>
-<wire x1="24.13" y1="19.05" x2="24.13" y2="43.18" width="0.6096" layer="16"/>
-<wire x1="73.66" y1="19.05" x2="24.13" y2="19.05" width="0.6096" layer="16"/>
-<wire x1="73.66" y1="16.51" x2="73.66" y2="19.05" width="0.6096" layer="16"/>
-<wire x1="73.66" y1="19.05" x2="73.66" y2="43.18" width="0.6096" layer="16"/>
 </signal>
 <signal name="S$9">
@@
 <vertex x="0" y="68.58"/>
 </polygon>
+<wire x1="66.04" y1="46.355" x2="66.04" y2="55.88" width="0.6096" layer="1"/>
+<wire x1="16.51" y1="48.26" x2="66.04" y2="48.26" width="0.6096" layer="16"/>
+<wire x1="16.51" y1="48.26" x2="16.51" y2="45.72" width="0.6096" layer="16"/>
+<wire x1="66.04" y1="48.26" x2="66.04" y2="45.72" width="0.6096" layer="16"/>
+<wire x1="66.04" y1="45.72" x2="66.04" y2="46.355" width="0" layer="19" extent="1-16"/>
 </signal>
 <signal name="S$11">
@@
 <wire x1="49.53" y1="39.37" x2="49.53" y2="62.23" width="0.6096" layer="1"/>
 </signal>
-<signal name="S$15">
+<signal name="VIN">
 <wire x1="68.58" y1="55.88" x2="68.58" y2="52.705" width="0.6096" layer="16"/>
 <wire x1="68.58" y1="52.705" x2="73.66" y2="52.705" width="0.6096" layer="16"/>
 <wire x1="73.66" y1="52.705" x2="73.66" y2="45.72" width="0.6096" layer="16"/>
+<wire x1="24.13" y1="16.51" x2="24.13" y2="19.05" width="0.6096" layer="16"/>
+<wire x1="24.13" y1="19.05" x2="24.13" y2="43.18" width="0.6096" layer="16"/>
+<wire x1="73.66" y1="19.05" x2="24.13" y2="19.05" width="0.6096" layer="16"/>
+<wire x1="73.66" y1="16.51" x2="73.66" y2="19.05" width="0.6096" layer="16"/>
+<wire x1="73.66" y1="19.05" x2="73.66" y2="43.18" width="0.6096" layer="16"/>
+<wire x1="73.66" y1="43.18" x2="73.66" y2="45.72" width="0" layer="19" extent="16-16"/>
 </signal>
 <signal name="S$21">
